File: DAS POWER/PCB/untitled.sch (EAGLE design)
At the start: 66 parts, among them J1 10118193-0001LF, J2 22-27-2041-04, Q1 12MHz, Q2 MMBT3904, Q3 MMBT3904, U1 CH340G, U2 AMS1117, U3 ESP32-WROOM-32D, X1 MSTBA2, X2 MSTBA6, X3 MSTBA6, X4 MSTBA6, X5 MSTBA2, X6 MSTBA2, X7 MSTBA2, X8 MSTBA2, X9 22-23-2021

Commit message: revisi final tanggal 21/02.2023
Parts:
- removed X1: MSTBA2, con-phoenix-508:MSTBA2
- removed X3: MSTBA6, con-phoenix-508:MSTBA6
- added X10: MSTBA9, con-phoenix-508:MSTBA9
Connections:
- removed net A0+: ADS1.A0, X3-6.1
- removed net A0-: ADS1.A1, X3-5.1
- removed net A1+: ADS1.A2, X3-4.1
- removed net A1-: ADS1.A3, X3-3.1
- removed net A2+: ADS2.A0, X3-2.1
- removed net A2-: ADS2.A1, X3-1.1
- removed net N$3: MINI1.IN+, X1-1.1
- removed net N$5: MINI1.IN-, X1-2.1
- new net +12V: MINI1.IN+, X10-2.1, X10-5.1, X10-8.1
- new net A0: ADS1.A2, X10-3.1
- new net A1: ADS1.A1, X10-6.1
- new net A2: ADS1.A0, X10-9.1
- net GND: now also MINI1.IN-, X10-1.1, X10-4.1, X10-7.1

Commit message: PCB DAS POWER
Connections:
- net OUT+: now also U$1.3V3, U$1.3V3.2
- net VCC: no longer U$1.3V3, U$1.3V3.2
Changed lines of the file:
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@@
 <part name="P+5" library="supply1" library_urn="urn:adsk.eagle:library:371" deviceset="VCC" device=""/>
 <part name="U$1" library="ethernet-mikroavr" deviceset="MINI_W5500" device=""/>
-<part name="P+6" library="supply1" library_urn="urn:adsk.eagle:library:371" deviceset="VCC" device=""/>
 <part name="GND7" library="supply1" library_urn="urn:adsk.eagle:library:371" deviceset="GND" device=""/>
 <part name="PZEM-DC1" library="pzem-dc" deviceset="PZEM-DC" device=""/>
@@
 </instance>
 <instance part="U$1" gate="G$1" x="93.98" y="137.16" smashed="yes"/>
-<instance part="P+6" gate="VCC" x="111.76" y="154.94" smashed="yes">
-<attribute name="VALUE" x="109.22" y="152.4" size="1.778" layer="96" rot="R90"/>
-</instance>
 <instance part="GND7" gate="1" x="66.04" y="147.32" smashed="yes">
 <attribute name="VALUE" x="63.5" y="144.78" size="1.778" layer="96"/>
@@
 <label x="40.64" y="99.06" size="0.6096" layer="95" xref="yes"/>
 </segment>
+<segment>
+<pinref part="U$1" gate="G$1" pin="3V3.2"/>
+<pinref part="U$1" gate="G$1" pin="3V3"/>
+<wire x1="106.68" y1="147.32" x2="106.68" y2="149.86" width="0.1524" layer="91"/>
+<wire x1="111.76" y1="149.86" x2="106.68" y2="149.86" width="0.1524" layer="91"/>
+<junction x="106.68" y="149.86"/>
+<label x="111.76" y="149.86" size="0.6096" layer="95" xref="yes"/>
+</segment>
 </net>
 <net name="VCC" class="0">
@@
 <pinref part="P+5" gate="VCC" pin="VCC"/>
 </segment>
-<segment>
-<pinref part="U$1" gate="G$1" pin="3V3.2"/>
-<pinref part="U$1" gate="G$1" pin="3V3"/>
-<wire x1="106.68" y1="147.32" x2="106.68" y2="149.86" width="0.1524" layer="91"/>
-<pinref part="P+6" gate="VCC" pin="VCC"/>
-<wire x1="111.76" y1="152.4" x2="111.76" y2="149.86" width="0.1524" layer="91"/>
-<wire x1="111.76" y1="149.86" x2="106.68" y2="149.86" width="0.1524" layer="91"/>
-<junction x="106.68" y="149.86"/>
-</segment>
-</net>
+</net>
